Commit message: Change joint controller type
Edited 'naoTransmission.xacro' and changed the type of each joint to effort_controller/
JointPositionController.

Changed the robot namespace to 'nao' and commented HipYaw Mimic plugin on 'naoGazebo.xacro'.

Commented the finger models on 'nao_robot.xacro'

File: nao_description/urdf/naoV40_generated_urdf/nao.urdf (robot description, URDF)
Before this commit: robot NaoH25V40, 83 links, 82 joints
Links:
- removed link CameraBottom_optical_frame
- removed link CameraTop_optical_frame
- removed link ChestButton_frame
- removed link Head
- removed link HeadTouchFront_frame
- removed link HeadTouchMiddle_frame
- removed link HeadTouchRear_frame
- removed link ImuTorsoAccelerometer_frame
- removed link ImuTorsoGyrometer_frame
- removed link LAnklePitch
- removed link LBicep
- removed link LElbow
- removed link LFinger11_link
- removed link LFinger12_link
- removed link LFinger13_link
- removed link LFinger21_link
- removed link LFinger22_link
- removed link LFinger23_link
- removed link LFootBumperLeft_frame
- removed link LFootBumperRight_frame
- removed link LForeArm
- removed link LFsrFL_frame
- removed link LFsrFR_frame
- removed link LFsrRL_frame
- removed link LFsrRR_frame
- removed link LHandTouchBack_frame
- removed link LHandTouchLeft_frame
- removed link LHandTouchRight_frame
- removed link LHip
- removed link LInfraRed_frame
- removed link LPelvis
- removed link LShoulder
- removed link LSonar_frame
- removed link LThigh
- removed link LThumb1_link
- removed link LThumb2_link
- removed link LTibia
- removed link MicroFrontCenter_frame
- removed link MicroRearCenter_frame
- removed link MicroSurroundLeft_frame
- removed link MicroSurroundRight_frame
- removed link Neck
- removed link RAnklePitch
- removed link RBicep
- removed link RElbow
- removed link RFinger11_link
- removed link RFinger12_link
- removed link RFinger13_link
- removed link RFinger21_link
- removed link RFinger22_link
- removed link RFinger23_link
- removed link RFootBumperLeft_frame
- removed link RFootBumperRight_frame
- removed link RForeArm
- removed link RFsrFL_frame
- removed link RFsrFR_frame
- removed link RFsrRL_frame
- removed link RFsrRR_frame
- removed link RHandTouchBack_frame
- removed link RHandTouchLeft_frame
- removed link RHandTouchRight_frame
- removed link RHip
- removed link RInfraRed_frame
- removed link RPelvis
- removed link RShoulder
- removed link RSonar_frame
- removed link RThigh
- removed link RThumb1_link
- removed link RThumb2_link
- removed link RTibia
- added link HeadPitch_link, mass 0.60533; visual cylinder length=0.14 radius=0.04
- added link HeadYaw_link, mass 0.06442
- added link LAnklePitch_link, mass 0.13415
- added link LAnkleRoll_link, mass 0.16178; visual cylinder length=0.046 radius=0.015
- added link LElbowRoll_link, mass 0.07778; visual cylinder length=0.05065 radius=0.015
- added link LElbowYaw_link, mass 0.06483
- added link LHipPitch_link, mass 0.38972; visual cylinder length=0.1 radius=0.015
- added link LHipRoll_link, mass 0.13053
- added link LHipYawPitch_link, mass 0.07050
- added link LKneePitch_link, mass 0.29152; visual cylinder length=0.1 radius=0.015
- added link LShoulderPitch_link, mass 0.07504
- added link LShoulderRoll_link, mass 0.15777; visual cylinder length=0.09 radius=0.015
- added link LWristYaw_link, mass 0.18533; visual cylinder length=0.058 radius=0.015
- added link RAnklePitch_link, mass 0.13415
- added link RAnkleRoll_link, mass 0.16178; visual cylinder length=0.046 radius=0.015
- added link RElbowRoll_link, mass 0.07778; visual cylinder length=0.05065 radius=0.015
- added link RElbowYaw_link, mass 0.06483
- added link RHipPitch_link, mass 0.38972; visual cylinder length=0.1 radius=0.015
- added link RHipRoll_link, mass 0.13053
- added link RHipYawPitch_link, mass 0.07050
- added link RKneePitch_link, mass 0.29152; visual cylinder length=0.1 radius=0.015
- added link RShoulderPitch_link, mass 0.07504
- added link RShoulderRoll_link, mass 0.15794; visual cylinder length=0.09 radius=0.015
- added link RWristYaw_link, mass 0.18533; visual cylinder length=0.058 radius=0.015
- link l_ankle: mass 0.16184 -> None; geometry 
- link l_gripper: mass 2e-06 -> None
- link l_sole: geometry visual box size=0.16 0.06 0.015
- link l_wrist: mass 0.18533 -> None; geometry 
- link r_ankle: mass 0.16184 -> None; geometry 
- link r_gripper: mass 2e-06 -> None
- link r_sole: geometry visual box size=0.16 0.06 0.015
- link r_wrist: mass 0.18533 -> None; geometry 
- link torso: geometry visual cylinder length=0.2115 radius=0.015
Joints:
- removed joint Accelerometer_sensor_fixedjoint
- removed joint CameraBottom_optical_frame_fixedjoint
- removed joint CameraBottom_sensor_fixedjoint
- removed joint CameraTop_optical_frame_fixedjoint
- removed joint CameraTop_sensor_fixedjoint
- removed joint ChestBoard/Button_sensor_fixedjoint
- removed joint Gyrometer_sensor_fixedjoint
- removed joint Head/Touch/Front_sensor_fixedjoint
- removed joint Head/Touch/Middle_sensor_fixedjoint
- removed joint Head/Touch/Rear_sensor_fixedjoint
- removed joint InfraredL_sensor_fixedjoint
- removed joint InfraredR_sensor_fixedjoint
- removed joint LFinger11
- removed joint LFinger12
- removed joint LFinger13
- removed joint LFinger21
- removed joint LFinger22
- removed joint LFinger23
- removed joint LFoot/Bumper/Left_sensor_fixedjoint
- removed joint LFoot/Bumper/Right_sensor_fixedjoint
- removed joint LFoot/FSR/FrontLeft_sensor_fixedjoint
- removed joint LFoot/FSR/FrontRight_sensor_fixedjoint
- removed joint LFoot/FSR/RearLeft_sensor_fixedjoint
- removed joint LFoot/FSR/RearRight_sensor_fixedjoint
- removed joint LHand
- removed joint LHand/Touch/Back_sensor_fixedjoint
- removed joint LHand/Touch/Left_sensor_fixedjoint
- removed joint LHand/Touch/Right_sensor_fixedjoint
- removed joint LLeg_effector_fixedjoint
- removed joint LThumb1
- removed joint LThumb2
- removed joint MicroFront_sensor_fixedjoint
- removed joint MicroLeft_sensor_fixedjoint
- removed joint MicroRear_sensor_fixedjoint
- removed joint MicroRight_sensor_fixedjoint
- removed joint RFinger11
- removed joint RFinger12
- removed joint RFinger13
- removed joint RFinger21
- removed joint RFinger22
- removed joint RFinger23
- removed joint RFoot/Bumper/Left_sensor_fixedjoint
- removed joint RFoot/Bumper/Right_sensor_fixedjoint
- removed joint RFoot/FSR/FrontLeft_sensor_fixedjoint
- removed joint RFoot/FSR/FrontRight_sensor_fixedjoint
- removed joint RFoot/FSR/RearLeft_sensor_fixedjoint
- removed joint RFoot/FSR/RearRight_sensor_fixedjoint
- removed joint RHand
- removed joint RHand/Touch/Back_sensor_fixedjoint
- removed joint RHand/Touch/Left_sensor_fixedjoint
- removed joint RHand/Touch/Right_sensor_fixedjoint
- removed joint RLeg_effector_fixedjoint
- removed joint RThumb1
- removed joint RThumb2
- removed joint Sonar/Left_sensor_fixedjoint
- removed joint Sonar/Right_sensor_fixedjoint
- removed joint base_link_fixedjoint
- added joint CameraBottom: type fixed, parent HeadPitch_link, child CameraBottom_frame, origin xyz=0.05071 0 0.01774 rpy=-2.263692 0 -1.5707963267948966
- added joint CameraTop: type fixed, parent HeadPitch_link, child CameraTop_frame, origin xyz=0.05871 0 0.06364 rpy=-1.59174 0 -1.5707963267948966
- added joint base_joint: type fixed, parent base_link, child torso, origin xyz=0 0 0 rpy=0 0 0
- added joint l_ankle_joint: type fixed, parent LAnkleRoll_link, child l_ankle, origin xyz=0 0 0
- added joint l_gripper_joint: type fixed, parent l_wrist, child l_gripper, origin xyz=0.058 0 -0.0159
- added joint l_sole_joint: type fixed, parent l_ankle, child l_sole, origin xyz=0 0 -0.04519
- added joint l_wrist_joint: type fixed, parent LWristYaw_link, child l_wrist, origin xyz=0 0 0
- added joint r_ankle_joint: type fixed, parent RAnkleRoll_link, child r_ankle, origin xyz=0 0 0
- added joint r_gripper_joint: type fixed, parent r_wrist, child r_gripper, origin xyz=0.058 0 -0.0159
- added joint r_sole_joint: type fixed, parent r_ankle, child r_sole, origin xyz=0 0 -0.04519
- added joint r_wrist_joint: type fixed, parent RWristYaw_link, child r_wrist, origin xyz=0 0 0
- joint HeadPitch: axis 0 1.0 0 -> 0 1 0; child Head -> HeadPitch_link; limit lower=-0.671952 upper=0.514872 effort=1.532 velocity=7.19407 -> lower=-0.6720 upper=0.5149 effort=30 velocity=3.0; parent Neck -> HeadYaw_link
- joint HeadYaw: axis 0 0 1.0 -> 0 0 1; child Neck -> HeadYaw_link; limit lower=-2.08567 upper=2.08567 effort=1.547 velocity=8.26797 -> lower=-2.0857 upper=2.0857 effort=30 velocity=3.0
- joint LAnklePitch: axis 0 1.0 0 -> 0 1 0; child LAnklePitch -> LAnklePitch_link; limit lower=-1.18944 upper=0.922581 effort=3.023 velocity=6.40239 -> lower=-1.186448 upper=0.922747 effort=30 velocity=3.0; origin xyz=0 0 -0.1029 rpy=0 0 0 -> xyz=0 0 -0.10290 rpy=0 0 0; parent LTibia -> LKneePitch_link
- joint LAnkleRoll: axis 1.0 0 0 -> 1 0 0; child l_ankle -> LAnkleRoll_link; limit lower=-0.397761 upper=0.768992 effort=3.348 velocity=4.16174 -> lower=-0.769001 upper=0.397880 effort=30 velocity=3.0; parent LAnklePitch -> LAnklePitch_link
- joint LElbowRoll: axis 0 0 1.0 -> 0 0 1; child LForeArm -> LElbowRoll_link; limit lower=-1.54462 upper=-0.0349066 effort=1.532 velocity=7.19407 -> lower=-1.5446 upper=-0.0349 effort=30 velocity=3.0; parent LElbow -> LElbowYaw_link
- joint LElbowYaw: axis 1.0 0 0 -> 1 0 0; child LElbow -> LElbowYaw_link; limit lower=-2.08567 upper=2.08567 effort=1.547 velocity=8.26797 -> lower=-2.0857 upper=2.0857 effort=30 velocity=3.0; parent LBicep -> LShoulderRoll_link
- joint LHipPitch: axis 0 1.0 0 -> 0 1 0; child LThigh -> LHipPitch_link; limit lower=-1.53589 upper=0.48398 effort=3.023 velocity=6.40239 -> lower=-1.772308 upper=0.484090 effort=30 velocity=3.0; parent LHip -> LHipRoll_link
- joint LHipRoll: axis 1.0 0 0 -> 1 0 0; child LHip -> LHipRoll_link; limit lower=-0.379435 upper=0.79046 effort=3.348 velocity=4.16174 -> lower=-0.379472 upper=0.790477 effort=30 velocity=3.0; parent LPelvis -> LHipYawPitch_link
- joint LHipYawPitch: child LPelvis -> LHipYawPitch_link; limit lower=-1.14529 upper=0.740718 effort=3.348 velocity=4.16174 -> lower=-1.145303 upper=0.740810 effort=30 velocity=3.0
- joint LKneePitch: axis 0 1.0 0 -> 0 1 0; child LTibia -> LKneePitch_link; limit lower=-0.0923279 upper=2.11255 effort=3.023 velocity=6.40239 -> lower=-0.092346 upper=2.112528 effort=30 velocity=3.0; parent LThigh -> LHipPitch_link
- joint LShoulderPitch: axis 0 1.0 0 -> 0 1 0; child LShoulder -> LShoulderPitch_link; limit lower=-2.08567 upper=2.08567 effort=1.329 velocity=8.26797 -> lower=-2.0857 upper=2.0857 effort=30 velocity=3.0
- joint LShoulderRoll: axis 0 0 1.0 -> 0 0 1; child LBicep -> LShoulderRoll_link; limit lower=-0.314159 upper=1.32645 effort=1.7835 velocity=7.19407 -> lower=-0.3142 upper=1.3265 effort=30 velocity=3.0; parent LShoulder -> LShoulderPitch_link
- joint LWristYaw: axis 1.0 0 0 -> 1 0 0; child l_wrist -> LWristYaw_link; limit lower=-1.82387 upper=1.82387 effort=0.4075 velocity=24.6229 -> lower=-1.8238 upper=1.8238 effort=30 velocity=3.0; parent LForeArm -> LElbowRoll_link
- joint RAnklePitch: axis 0 1.0 0 -> 0 1 0; child RAnklePitch -> RAnklePitch_link; limit lower=-1.1863 upper=0.932006 effort=3.0226 velocity=6.40239 -> lower=-1.186448 upper=0.922747 effort=30 velocity=3.0; origin xyz=0 0 -0.1029 rpy=0 0 0 -> xyz=0 0 -0.10290 rpy=0 0 0; parent RTibia -> RKneePitch_link
- joint RAnkleRoll: axis 1.0 0 0 -> 1 0 0; child r_ankle -> RAnkleRoll_link; limit lower=-0.768992 upper=0.397761 effort=3.348 velocity=4.16174 -> lower=-0.388676 upper=0.785875 effort=30 velocity=3.0; parent RAnklePitch -> RAnklePitch_link
- joint RElbowRoll: axis 0 0 1.0 -> 0 0 1; child RForeArm -> RElbowRoll_link; limit lower=0.0349066 upper=1.54462 effort=1.532 velocity=7.19407 -> lower=0.0349 upper=1.5446 effort=30 velocity=3.0; parent RElbow -> RElbowYaw_link
- joint RElbowYaw: axis 1.0 0 0 -> 1 0 0; child RElbow -> RElbowYaw_link; limit lower=-2.08567 upper=2.08567 effort=1.547 velocity=8.26797 -> lower=-2.0857 upper=2.0857 effort=30 velocity=3.0; parent RBicep -> RShoulderRoll_link
- joint RHipPitch: axis 0 1.0 0 -> 0 1 0; child RThigh -> RHipPitch_link; limit lower=-1.53589 upper=0.48398 effort=3.0226 velocity=6.40239 -> lower=-1.772308 upper=0.484090 effort=30 velocity=3.0; parent RHip -> RHipRoll_link
- joint RHipRoll: axis 1.0 0 0 -> 1 0 0; child RHip -> RHipRoll_link; limit lower=-0.79046 upper=0.379435 effort=3.348 velocity=4.16174 -> lower=-0.738321 upper=0.414754 effort=30 velocity=3.0; parent RPelvis -> RHipYawPitch_link
- joint RHipYawPitch: child RPelvis -> RHipYawPitch_link; limit lower=-1.14529 upper=0.740718 effort=3.348 velocity=4.16174 -> lower=-1.145303 upper=0.740810 effort=30 velocity=3.0; mimic joint=LHipYawPitch multiplier=1.0 offset=0 -> joint=LHipYawPitch multiplier=1 offset=0
- joint RKneePitch: axis 0 1.0 0 -> 0 1 0; child RTibia -> RKneePitch_link; limit lower=-0.0923279 upper=2.11255 effort=3.0226 velocity=6.40239 -> lower=-0.092346 upper=2.112528 effort=30 velocity=3.0; parent RThigh -> RHipPitch_link
- joint RShoulderPitch: axis 0 1.0 0 -> 0 1 0; child RShoulder -> RShoulderPitch_link; limit lower=-2.08567 upper=2.08567 effort=1.329 velocity=8.26797 -> lower=-2.0857 upper=2.0857 effort=30 velocity=3.0
- joint RShoulderRoll: axis 0 0 1.0 -> 0 0 1; child RBicep -> RShoulderRoll_link; limit lower=-1.32645 upper=0.314159 effort=1.783 velocity=7.19407 -> lower=-1.3265 upper=0.3142 effort=30 velocity=3.0; parent RShoulder -> RShoulderPitch_link
- joint RWristYaw: axis 1.0 0 0 -> 1 0 0; child r_wrist -> RWristYaw_link; limit lower=-1.82387 upper=1.82387 effort=0.4075 velocity=24.6229 -> lower=-1.8238 upper=1.8238 effort=30 velocity=3.0; parent RForeArm -> RElbowRoll_link
- joint gaze_joint: origin xyz=0.05871 0 0.06364 rpy=0 0 0 -> xyz=0.0539 0 0.05; parent Head -> HeadPitch_link

File: nao_description/urdf/naoV40_generated_urdf/naoGazebo.xacro (robot description, xacro)
@@ -72,5 +72,5 @@
     <gazebo>
         <plugin filename="libgazebo_ros_control.so" name="gazebo_ros_control">
-            <robotNamespace></robotNamespace>
+            <robotNamespace>nao</robotNamespace>
             <robotSimType>gazebo_ros_control/DefaultRobotHWSim</robotSimType>
         </plugin>
@@ -90,5 +90,5 @@
         </plugin>
 -->
-<!--        <plugin name="gazebo_ros_imu_controller" filename="${imu_plugin}">
+<!--         <plugin name="gazebo_ros_imu_controller" filename="${imu_plugin}">
             <robotNamespace>/nao_dcm</robotNamespace>
             <topicName>imu_data</topicName>
@@ -103,12 +103,12 @@
             <updateRate>30.0</updateRate>
             <alwaysOn>true</alwaysOn>
-        </plugin>
--->        <!-- Mimic joints through plugin develop by costashatz based on implementation by Goncalo Cabrita -->
-        <plugin name="mimic_hipyawpitch" filename="libroboticsgroup_gazebo_mimic_joint_plugin.so">
+        </plugin> -->
+        <!-- Mimic joints through plugin develop by costashatz based on implementation by Goncalo Cabrita -->
+<!--         <plugin name="mimic_hipyawpitch" filename="libroboticsgroup_gazebo_mimic_joint_plugin.so">
             <joint>LHipYawPitch</joint>
             <mimicJoint>RHipYawPitch</mimicJoint>
             <multiplier>1.0</multiplier>
             <offset>0.0</offset>
-        </plugin>
+        </plugin> -->
         <xacro:FingerMimics side="L" num="1"/>
         <xacro:FingerMimics side="L" num="2"/>
