Commit message: Change joint controller type
Edited 'naoTransmission.xacro' and changed the type of each joint to effort_controller/
JointPositionController.

Changed the robot namespace to 'nao' and commented HipYaw Mimic plugin on 'naoGazebo.xacro'.

Commented the finger models on 'nao_robot.xacro'

File: nao_description/urdf/naoV40_generated_urdf/naoTransmission.xacro (robot description, xacro)
@@ -12,9 +12,9 @@
 		<type>transmission_interface/SimpleTransmission</type>
 		<joint name="HeadYaw">
-        	<hardwareInterface>PositionJointInterface</hardwareInterface>
+        	<hardwareInterface>hardware_interface/EffortJointInterface</hardwareInterface>
 		</joint>
         <actuator name="HeadYaw_Motor">
 			<!-- Dummy Values -->
-			<hardwareInterface>PositionJointInterface</hardwareInterface>
+			<hardwareInterface>hardware_interface/EffortJointInterface</hardwareInterface>
 			<mechanicalReduction>${speed_red_type3A}</mechanicalReduction>
 		</actuator>
@@ -23,9 +23,9 @@
 		<type>transmission_interface/SimpleTransmission</type>
 		<joint name="HeadPitch">
-            <hardwareInterface>PositionJointInterface</hardwareInterface>
+            <hardwareInterface>hardware_interface/EffortJointInterface</hardwareInterface>
         </joint>
 		<actuator name="HeadPitch_Motor">
 			<!-- Dummy Values -->
-			<hardwareInterface>PositionJointInterface</hardwareInterface>
+			<hardwareInterface>hardware_interface/EffortJointInterface</hardwareInterface>
 			<mechanicalReduction>${speed_red_type3B}</mechanicalReduction>
 		</actuator>
@@ -37,8 +37,8 @@
 			<type>transmission_interface/SimpleTransmission</type>
 			<joint name="${side}ShoulderPitch">
-              <hardwareInterface>PositionJointInterface</hardwareInterface>
+              <hardwareInterface>hardware_interface/EffortJointInterface</hardwareInterface>
             </joint>
 			<actuator name="${side}ShoulderPitch_Motor">
-				<hardwareInterface>PositionJointInterface</hardwareInterface>
+				<hardwareInterface>hardware_interface/EffortJointInterface</hardwareInterface>
 				<mechanicalReduction>${speed_red_type3A}</mechanicalReduction>
 			</actuator>
@@ -47,8 +47,8 @@
 			<type>transmission_interface/SimpleTransmission</type>
 			<joint name="${side}ShoulderRoll">
-     			<hardwareInterface>PositionJointInterface</hardwareInterface>
+     			<hardwareInterface>hardware_interface/EffortJointInterface</hardwareInterface>
             </joint>
 			<actuator name="${side}ShoulderRoll_Motor">
-				<hardwareInterface>PositionJointInterface</hardwareInterface>
+				<hardwareInterface>hardware_interface/EffortJointInterface</hardwareInterface>
 				<mechanicalReduction>${speed_red_type3B}</mechanicalReduction>
 			</actuator>
@@ -57,8 +57,8 @@
 			<type>transmission_interface/SimpleTransmission</type>
 			<joint name="${side}ElbowYaw">
-              <hardwareInterface>PositionJointInterface</hardwareInterface>
+              <hardwareInterface>hardware_interface/EffortJointInterface</hardwareInterface>
             </joint>
 			<actuator name="${side}ElbowYaw_Motor">
-				<hardwareInterface>PositionJointInterface</hardwareInterface>
+				<hardwareInterface>hardware_interface/EffortJointInterface</hardwareInterface>
 				<mechanicalReduction>${speed_red_type3A}</mechanicalReduction>
 			</actuator>
@@ -67,8 +67,8 @@
 			<type>transmission_interface/SimpleTransmission</type>
 			<joint name="${side}ElbowRoll">
-    			<hardwareInterface>PositionJointInterface</hardwareInterface>
+    			<hardwareInterface>hardware_interface/EffortJointInterface</hardwareInterface>
             </joint>
 			<actuator name="${side}ElbowRoll_Motor">
-				<hardwareInterface>PositionJointInterface</hardwareInterface>
+				<hardwareInterface>hardware_interface/EffortJointInterface</hardwareInterface>
 				<mechanicalReduction>${speed_red_type3B}</mechanicalReduction>
 			</actuator>
@@ -77,8 +77,8 @@
 			<type>transmission_interface/SimpleTransmission</type>
 			<joint name="${side}WristYaw">
-              <hardwareInterface>PositionJointInterface</hardwareInterface>
+              <hardwareInterface>hardware_interface/EffortJointInterface</hardwareInterface>
             </joint>
 			<actuator name="${side}WristYaw_Motor">
-				<hardwareInterface>PositionJointInterface</hardwareInterface>
+				<hardwareInterface>hardware_interface/EffortJointInterface</hardwareInterface>
 				<mechanicalReduction>${speed_red_type2A}</mechanicalReduction>
 			</actuator>
@@ -87,8 +87,8 @@
 			<type>transmission_interface/SimpleTransmission</type>
 			<joint name="${side}Hand">
-  			  <hardwareInterface>PositionJointInterface</hardwareInterface>
+  			  <hardwareInterface>hardware_interface/EffortJointInterface</hardwareInterface>
             </joint>
 			<actuator name="${side}Hand_Motor">
-				<hardwareInterface>PositionJointInterface</hardwareInterface>
+				<hardwareInterface>hardware_interface/EffortJointInterface</hardwareInterface>
 				<mechanicalReduction>${speed_red_type2B}</mechanicalReduction>
 			</actuator>
@@ -103,9 +103,9 @@
 			<type>transmission_interface/SimpleTransmission</type>
 			<joint name="${side}HipYawPitch">
-    			<hardwareInterface>PositionJointInterface</hardwareInterface>
+    			<hardwareInterface>hardware_interface/EffortJointInterface</hardwareInterface>
             </joint>
 			<actuator name="${side}HipYawPitch_Motor">
 				<!-- Dummy Values -->
-				<hardwareInterface>PositionJointInterface</hardwareInterface>
+				<hardwareInterface>hardware_interface/EffortJointInterface</hardwareInterface>
 				<mechanicalReduction>${speed_red_type1A}</mechanicalReduction>
 			</actuator>
@@ -114,9 +114,9 @@
 			<type>transmission_interface/SimpleTransmission</type>
 			<joint name="${side}HipRoll">
-			  <hardwareInterface>PositionJointInterface</hardwareInterface>
+			  <hardwareInterface>hardware_interface/EffortJointInterface</hardwareInterface>
             </joint>
 			<actuator name="${side}HipRoll_Motor">
 				<!-- Dummy Values -->
-				<hardwareInterface>PositionJointInterface</hardwareInterface>
+				<hardwareInterface>hardware_interface/EffortJointInterface</hardwareInterface>
 				<mechanicalReduction>${speed_red_type1A}</mechanicalReduction>
 			</actuator>
@@ -125,9 +125,9 @@
 			<type>transmission_interface/SimpleTransmission</type>
 			<joint name="${side}HipPitch">
-			  <hardwareInterface>PositionJointInterface</hardwareInterface>
+			  <hardwareInterface>hardware_interface/EffortJointInterface</hardwareInterface>
             </joint>
 			<actuator name="${side}HipPitch_Motor">
 				<!-- Dummy Values -->
-				<hardwareInterface>PositionJointInterface</hardwareInterface>
+				<hardwareInterface>hardware_interface/EffortJointInterface</hardwareInterface>
 				<mechanicalReduction>${speed_red_type1B}</mechanicalReduction>
 			</actuator>
@@ -136,9 +136,9 @@
 			<type>transmission_interface/SimpleTransmission</type>
 			<joint name="${side}KneePitch">
-       			<hardwareInterface>PositionJointInterface</hardwareInterface>
+       			<hardwareInterface>hardware_interface/EffortJointInterface</hardwareInterface>
             </joint>
 			<actuator name="${side}KneePitch_Motor">
 				<!-- Dummy Values -->
-				<hardwareInterface>PositionJointInterface</hardwareInterface>
+				<hardwareInterface>hardware_interface/EffortJointInterface</hardwareInterface>
 				<mechanicalReduction>${speed_red_type1B}</mechanicalReduction>
 			</actuator>
@@ -147,9 +147,9 @@
 			<type>transmission_interface/SimpleTransmission</type>
 			<joint name="${side}AnklePitch">
-  			  <hardwareInterface>PositionJointInterface</hardwareInterface>
+  			  <hardwareInterface>hardware_interface/EffortJointInterface</hardwareInterface>
             </joint>
 			<actuator name="${side}AnklePitch_Motor">
 				<!-- Dummy Values -->
-				<hardwareInterface>PositionJointInterface</hardwareInterface>
+				<hardwareInterface>hardware_interface/EffortJointInterface</hardwareInterface>
 				<mechanicalReduction>${speed_red_type1B}</mechanicalReduction>
 			</actuator>
@@ -158,9 +158,9 @@
 			<type>transmission_interface/SimpleTransmission</type>
 			<joint name="${side}AnkleRoll">
-      			<hardwareInterface>PositionJointInterface</hardwareInterface>
+      			<hardwareInterface>hardware_interface/EffortJointInterface</hardwareInterface>
             </joint>
 			<actuator name="${side}AnkleRoll_Motor">
 				<!-- Dummy Values -->
-				<hardwareInterface>PositionJointInterface</hardwareInterface>
+				<hardwareInterface>hardware_interface/EffortJointInterface</hardwareInterface>
 				<mechanicalReduction>${speed_red_type1A}</mechanicalReduction>
 			</actuator>

File: nao_description/urdf/naoV40_generated_urdf/nao_robot.xacro (robot description, xacro)
@@ -10,5 +10,5 @@
 	<xacro:include filename="nao_arms.xacro"/>
 	<xacro:include filename="nao_sensors.xacro"/>
-	<xacro:include filename="nao_fingers.xacro"/>
+	<!-- <xacro:include filename="nao_fingers.xacro"/> -->
 	<xacro:include filename="naoGazebo.xacro"/>
 	<xacro:include filename="naoTransmission.xacro"/>
