Commit message: Fix FSR link collision names
Changed the name of the collision tags on the .xacro files for Gazebo
simulation on 'naoGazebo.xacro', which did not match the actual collision
names due to a known sdformat bug (Issue #113).

File: nao_description/urdf/naoV40_generated_urdf/nao.urdf (robot description, URDF)
Before this commit: robot nao, 37 links, 36 joints
Links:
- removed link HeadPitch_link
- removed link HeadYaw_link
- removed link LAnklePitch_link
- removed link LAnkleRoll_link
- removed link LElbowRoll_link
- removed link LElbowYaw_link
- removed link LHipPitch_link
- removed link LHipRoll_link
- removed link LHipYawPitch_link
- removed link LKneePitch_link
- removed link LShoulderPitch_link
- removed link LShoulderRoll_link
- removed link LWristYaw_link
- removed link RAnklePitch_link
- removed link RAnkleRoll_link
- removed link RElbowRoll_link
- removed link RElbowYaw_link
- removed link RHipPitch_link
- removed link RHipRoll_link
- removed link RHipYawPitch_link
- removed link RKneePitch_link
- removed link RShoulderPitch_link
- removed link RShoulderRoll_link
- removed link RWristYaw_link
- added link CameraBottom_optical_frame
- added link CameraTop_optical_frame
- added link ChestButton_frame
- added link Head, mass 0.60533; collision mesh filename=package://nao_meshes/meshes/V40/HeadPitch_0.10.stl scale=0.1 0.1 0.1; visual mesh filename=package://nao_meshes/meshes/V40/HeadPitch.dae scale=0.1 0.1 0.1
- added link HeadTouchFront_frame
- added link HeadTouchMiddle_frame
- added link HeadTouchRear_frame
- added link ImuTorsoAccelerometer_frame
- added link ImuTorsoGyrometer_frame
- added link LAnklePitch, mass 0.13416; collision mesh filename=package://nao_meshes/meshes/V40/LAnklePitch_0.10.stl scale=0.1 0.1 0.1; visual mesh filename=package://nao_meshes/meshes/V40/LAnklePitch.dae scale=0.1 0.1 0.1
- added link LBicep, mass 0.15777; collision mesh filename=package://nao_meshes/meshes/V40/LShoulderRoll_0.10.stl scale=0.1 0.1 0.1; visual mesh filename=package://nao_meshes/meshes/V40/LShoulderRoll.dae scale=0.1 0.1 0.1
- added link LElbow, mass 0.06483
- added link LFootBumperLeft_frame
- added link LFootBumperRight_frame
- added link LForeArm, mass 0.07761; collision mesh filename=package://nao_meshes/meshes/V40/LElbowRoll_0.10.stl scale=0.1 0.1 0.1; visual mesh filename=package://nao_meshes/meshes/V40/LElbowRoll.dae scale=0.1 0.1 0.1
- added link LFsrFL_frame, mass 2e-06; collision box size=0.01 0.01 0.005
- added link LFsrFR_frame, mass 2e-06; collision box size=0.01 0.01 0.005
- added link LFsrRL_frame, mass 2e-06; collision box size=0.01 0.01 0.005
- added link LFsrRR_frame, mass 2e-06; collision box size=0.01 0.01 0.005
- added link LHandTouchBack_frame
- added link LHandTouchLeft_frame
- added link LHandTouchRight_frame
- added link LHip, mass 0.13053; collision mesh filename=package://nao_meshes/meshes/V40/LHipRoll_0.10.stl scale=0.1 0.1 0.1; visual mesh filename=package://nao_meshes/meshes/V40/LHipRoll.dae scale=0.1 0.1 0.1
- added link LInfraRed_frame
- added link LPelvis, mass 0.06981; collision mesh filename=package://nao_meshes/meshes/V40/LHipYawPitch_0.10.stl scale=0.1 0.1 0.1; visual mesh filename=package://nao_meshes/meshes/V40/LHipYawPitch.dae scale=0.1 0.1 0.1
- added link LShoulder, mass 0.07504; collision mesh filename=package://nao_meshes/meshes/V40/LShoulderPitch_0.10.stl scale=0.1 0.1 0.1; visual mesh filename=package://nao_meshes/meshes/V40/LShoulderPitch.dae scale=0.1 0.1 0.1
- added link LSonar_frame
- added link LThigh, mass 0.38968; collision mesh filename=package://nao_meshes/meshes/V40/LHipPitch_0.10.stl scale=0.1 0.1 0.1; visual mesh filename=package://nao_meshes/meshes/V40/LHipPitch.dae scale=0.1 0.1 0.1
- added link LTibia, mass 0.29142; collision mesh filename=package://nao_meshes/meshes/V40/LKneePitch_0.10.stl scale=0.1 0.1 0.1; visual mesh filename=package://nao_meshes/meshes/V40/LKneePitch.dae scale=0.1 0.1 0.1
- added link MicroFrontCenter_frame
- added link MicroRearCenter_frame
- added link MicroSurroundLeft_frame
- added link MicroSurroundRight_frame
- added link Neck, mass 0.06442; collision mesh filename=package://nao_meshes/meshes/V40/HeadYaw_0.10.stl scale=0.1 0.1 0.1; visual mesh filename=package://nao_meshes/meshes/V40/HeadYaw.dae scale=0.1 0.1 0.1
- added link RAnklePitch, mass 0.13416; collision mesh filename=package://nao_meshes/meshes/V40/RAnklePitch_0.10.stl scale=0.1 0.1 0.1; visual mesh filename=package://nao_meshes/meshes/V40/RAnklePitch.dae scale=0.1 0.1 0.1
- added link RBicep, mass 0.15777; collision mesh filename=package://nao_meshes/meshes/V40/RShoulderRoll_0.10.stl scale=0.1 0.1 0.1; visual mesh filename=package://nao_meshes/meshes/V40/RShoulderRoll.dae scale=0.1 0.1 0.1
- added link RElbow, mass 0.06483
- added link RFootBumperLeft_frame
- added link RFootBumperRight_frame
- added link RForeArm, mass 0.07761; collision mesh filename=package://nao_meshes/meshes/V40/RElbowRoll_0.10.stl scale=0.1 0.1 0.1; visual mesh filename=package://nao_meshes/meshes/V40/RElbowRoll.dae scale=0.1 0.1 0.1
- added link RFsrFL_frame, mass 2e-06; collision box size=0.01 0.01 0.005
- added link RFsrFR_frame, mass 2e-06; collision box size=0.01 0.01 0.005
- added link RFsrRL_frame, mass 2e-06; collision box size=0.01 0.01 0.005
- added link RFsrRR_frame, mass 2e-06; collision box size=0.01 0.01 0.005
- added link RHandTouchBack_frame
- added link RHandTouchLeft_frame
- added link RHandTouchRight_frame
- added link RHip, mass 0.13053; collision mesh filename=package://nao_meshes/meshes/V40/RHipRoll_0.10.stl scale=0.1 0.1 0.1; visual mesh filename=package://nao_meshes/meshes/V40/RHipRoll.dae scale=0.1 0.1 0.1
- added link RInfraRed_frame
- added link RPelvis, mass 0.06981; collision mesh filename=package://nao_meshes/meshes/V40/RHipYawPitch_0.10.stl scale=0.1 0.1 0.1; visual mesh filename=package://nao_meshes/meshes/V40/RHipYawPitch.dae scale=0.1 0.1 0.1
- added link RShoulder, mass 0.07504; collision mesh filename=package://nao_meshes/meshes/V40/RShoulderPitch_0.10.stl scale=0.1 0.1 0.1; visual mesh filename=package://nao_meshes/meshes/V40/RShoulderPitch.dae scale=0.1 0.1 0.1
- added link RSonar_frame
- added link RThigh, mass 0.38968; collision mesh filename=package://nao_meshes/meshes/V40/RHipPitch_0.10.stl scale=0.1 0.1 0.1; visual mesh filename=package://nao_meshes/meshes/V40/RHipPitch.dae scale=0.1 0.1 0.1
- added link RTibia, mass 0.29142; collision mesh filename=package://nao_meshes/meshes/V40/RKneePitch_0.10.stl scale=0.1 0.1 0.1; visual mesh filename=package://nao_meshes/meshes/V40/RKneePitch.dae scale=0.1 0.1 0.1
- link l_ankle: mass None -> 0.16184; geometry collision mesh filename=package://nao_meshes/meshes/V40/LAnkleRoll_0.10.stl scale=0.1 0.1 0.1; visual mesh filename=package://nao_meshes/meshes/V40/LAnkleRoll.dae scale=0.1 0.1 0.1
- link l_gripper: mass None -> 2e-06
- link l_sole: geometry 
- link l_wrist: mass None -> 0.18533; geometry collision mesh filename=package://nao_meshes/meshes/V40/LWristYaw_0.10.stl scale=0.1 0.1 0.1; visual mesh filename=package://nao_meshes/meshes/V40/LWristYaw.dae scale=0.1 0.1 0.1
- link r_ankle: mass None -> 0.16184; geometry collision mesh filename=package://nao_meshes/meshes/V40/RAnkleRoll_0.10.stl scale=0.1 0.1 0.1; visual mesh filename=package://nao_meshes/meshes/V40/RAnkleRoll.dae scale=0.1 0.1 0.1
- link r_gripper: mass None -> 2e-06
- link r_sole: geometry 
- link r_wrist: mass None -> 0.18533; geometry collision mesh filename=package://nao_meshes/meshes/V40/RWristYaw_0.10.stl scale=0.1 0.1 0.1; visual mesh filename=package://nao_meshes/meshes/V40/RWristYaw.dae scale=0.1 0.1 0.1
- link torso: geometry collision mesh filename=package://nao_meshes/meshes/V40/Torso_0.10.stl scale=0.1 0.1 0.1; visual mesh filename=package://nao_meshes/meshes/V40/Torso.dae scale=0.1 0.1 0.1
Joints:
- removed joint CameraBottom
- removed joint CameraTop
- removed joint base_joint
- removed joint l_ankle_joint
- removed joint l_gripper_joint
- removed joint l_sole_joint
- removed joint l_wrist_joint
- removed joint r_ankle_joint
- removed joint r_gripper_joint
- removed joint r_sole_joint
- removed joint r_wrist_joint
- added joint Accelerometer_sensor_fixedjoint: type fixed, parent torso, child ImuTorsoAccelerometer_frame, origin xyz=-0.008 0.00606 0.027 rpy=0 0 0, axis 0 0 0
- added joint CameraBottom_optical_frame_fixedjoint: type fixed, parent CameraBottom_frame, child CameraBottom_optical_frame, origin xyz=0 0 0 rpy=-1.57079632679 0 -1.57079632679
- added joint CameraBottom_sensor_fixedjoint: type fixed, parent Head, child CameraBottom_frame, origin xyz=0.05071 0 0.01774 rpy=0 0.692896 0, axis 0 0 0
- added joint CameraTop_optical_frame_fixedjoint: type fixed, parent CameraTop_frame, child CameraTop_optical_frame, origin xyz=0 0 0 rpy=-1.57079632679 0 -1.57079632679
- added joint CameraTop_sensor_fixedjoint: type fixed, parent Head, child CameraTop_frame, origin xyz=0.05871 0 0.06364 rpy=0 0.0209435 0, axis 0 0 0
- added joint ChestBoard/Button_sensor_fixedjoint: type fixed, parent torso, child ChestButton_frame, origin xyz=0.049871 0.001588 0.055163 rpy=0 0 0, axis 0 0 0
- added joint Gyrometer_sensor_fixedjoint: type fixed, parent torso, child ImuTorsoGyrometer_frame, origin xyz=-0.008 0.006 0.029 rpy=0 0 0, axis 0 0 0
- added joint Head/Touch/Front_sensor_fixedjoint: type fixed, parent Head, child HeadTouchFront_frame, origin xyz=0.0312 0 0.1014 rpy=0 -1.1861 0, axis 0 0 0
- added joint Head/Touch/Middle_sensor_fixedjoint: type fixed, parent Head, child HeadTouchMiddle_frame, origin xyz=0.001 0 0.1099 rpy=3.14159 -1.57079 -3.14159, axis 0 0 0
- added joint Head/Touch/Rear_sensor_fixedjoint: type fixed, parent Head, child HeadTouchRear_frame, origin xyz=-0.0257 0 0.1045 rpy=3.14159 -1.33319 -3.14159, axis 0 0 0
- added joint InfraredL_sensor_fixedjoint: type fixed, parent Head, child LInfraRed_frame, origin xyz=0.0441 0.0257 0.0466 rpy=0 0 0, axis 0 0 0
- added joint InfraredR_sensor_fixedjoint: type fixed, parent Head, child RInfraRed_frame, origin xyz=0.0441 -0.0257 0.0466 rpy=0 0 0, axis 0 0 0
- added joint LFoot/Bumper/Left_sensor_fixedjoint: type fixed, parent l_ankle, child LFootBumperLeft_frame, origin xyz=0.0876 0.019 -0.0353 rpy=0 0 0, axis 0 0 0
- added joint LFoot/Bumper/Right_sensor_fixedjoint: type fixed, parent l_ankle, child LFootBumperRight_frame, origin xyz=0.0876 -0.014 -0.0353 rpy=0 0 0, axis 0 0 0
- added joint LFoot/FSR/FrontLeft_sensor_fixedjoint: type fixed, parent l_ankle, child LFsrFL_frame, origin xyz=0.07025 0.0299 -0.04511 rpy=0 0 0, axis 0 0 0
- added joint LFoot/FSR/FrontRight_sensor_fixedjoint: type fixed, parent l_ankle, child LFsrFR_frame, origin xyz=0.07025 -0.0231 -0.04511 rpy=0 0 0, axis 0 0 0
- added joint LFoot/FSR/RearLeft_sensor_fixedjoint: type fixed, parent l_ankle, child LFsrRL_frame, origin xyz=-0.03025 0.0299 -0.04511 rpy=0 0 0, axis 0 0 0
- added joint LFoot/FSR/RearRight_sensor_fixedjoint: type fixed, parent l_ankle, child LFsrRR_frame, origin xyz=-0.02965 -0.0191 -0.04511 rpy=0 0 0, axis 0 0 0
- added joint LHand: type revolute, parent l_wrist, child l_gripper, origin xyz=0.05775 0 -0.01231 rpy=0 0 0, axis 1.0 0 0, limit lower=0 upper=1.0 effort=0.292 velocity=8.33
- added joint LHand/Touch/Back_sensor_fixedjoint: type fixed, parent l_wrist, child LHandTouchBack_frame, origin xyz=0.038 0 0.025 rpy=3.14159 -1.5708 3.14159, axis 0 0 0
- added joint LHand/Touch/Left_sensor_fixedjoint: type fixed, parent l_wrist, child LHandTouchLeft_frame, origin xyz=0.032 0.025 0.003 rpy=0 0 1.5708, axis 0 0 0
- added joint LHand/Touch/Right_sensor_fixedjoint: type fixed, parent l_wrist, child LHandTouchRight_frame, origin xyz=0.035 -0.025 0.0035 rpy=0 0 -1.5708, axis 0 0 0
- added joint LLeg_effector_fixedjoint: type fixed, parent l_ankle, child l_sole, origin xyz=0 0 -0.04511 rpy=0 0 0, axis 0 0 0
- added joint MicroFront_sensor_fixedjoint: type fixed, parent Head, child MicroFrontCenter_frame, origin xyz=0.041 0 0.091 rpy=0 0 0, axis 0 0 0
- added joint MicroLeft_sensor_fixedjoint: type fixed, parent Head, child MicroSurroundLeft_frame, origin xyz=-0.0195 0.0606 0.0331 rpy=0 0 0, axis 0 0 0
- added joint MicroRear_sensor_fixedjoint: type fixed, parent Head, child MicroRearCenter_frame, origin xyz=-0.0577 0 0.0693 rpy=0 0 0, axis 0 0 0
- added joint MicroRight_sensor_fixedjoint: type fixed, parent Head, child MicroSurroundRight_frame, origin xyz=-0.0195 -0.0606 0.0331 rpy=0 0 0, axis 0 0 0
- added joint RFoot/Bumper/Left_sensor_fixedjoint: type fixed, parent r_ankle, child RFootBumperLeft_frame, origin xyz=0.0876 0.014 -0.0353 rpy=0 0 0, axis 0 0 0
- added joint RFoot/Bumper/Right_sensor_fixedjoint: type fixed, parent r_ankle, child RFootBumperRight_frame, origin xyz=0.0876 -0.019 -0.0353 rpy=0 0 0, axis 0 0 0
- added joint RFoot/FSR/FrontLeft_sensor_fixedjoint: type fixed, parent r_ankle, child RFsrFL_frame, origin xyz=0.07025 0.0231 -0.04511 rpy=0 0 0, axis 0 0 0
- added joint RFoot/FSR/FrontRight_sensor_fixedjoint: type fixed, parent r_ankle, child RFsrFR_frame, origin xyz=0.07025 -0.0299 -0.04511 rpy=0 0 0, axis 0 0 0
- added joint RFoot/FSR/RearLeft_sensor_fixedjoint: type fixed, parent r_ankle, child RFsrRL_frame, origin xyz=-0.03025 0.0191 -0.04511 rpy=0 0 0, axis 0 0 0
- added joint RFoot/FSR/RearRight_sensor_fixedjoint: type fixed, parent r_ankle, child RFsrRR_frame, origin xyz=-0.02965 -0.0299 -0.04511 rpy=0 0 0, axis 0 0 0
- added joint RHand: type revolute, parent r_wrist, child r_gripper, origin xyz=0.05775 0 -0.01231 rpy=0 0 0, axis 1.0 0 0, limit lower=0 upper=1.0 effort=0.292 velocity=8.33
- added joint RHand/Touch/Back_sensor_fixedjoint: type fixed, parent r_wrist, child RHandTouchBack_frame, origin xyz=0.038 0 0.025 rpy=3.14159 -1.5708 3.14159, axis 0 0 0
- added joint RHand/Touch/Left_sensor_fixedjoint: type fixed, parent r_wrist, child RHandTouchLeft_frame, origin xyz=0.032 0.025 0.003 rpy=0 0 1.5708, axis 0 0 0
- added joint RHand/Touch/Right_sensor_fixedjoint: type fixed, parent r_wrist, child RHandTouchRight_frame, origin xyz=0.035 -0.025 0.0035 rpy=0 0 -1.5708, axis 0 0 0
- added joint RLeg_effector_fixedjoint: type fixed, parent r_ankle, child r_sole, origin xyz=0 0 -0.04511 rpy=0 0 0, axis 0 0 0
- added joint Sonar/Left_sensor_fixedjoint: type fixed, parent torso, child LSonar_frame, origin xyz=0.00558253 0.0192068 0.0623853 rpy=-0.00478508 0.0436497 0.392441, axis 0 0 0
- added joint Sonar/Right_sensor_fixedjoint: type fixed, parent torso, child RSonar_frame, origin xyz=0.00558253 -0.0192068 0.0623853 rpy=0.00478508 0.0436497 -0.392441, axis 0 0 0
- added joint base_link_fixedjoint: type fixed, parent base_link, child torso, origin xyz=0 0 0 rpy=0 0 0, axis 0 0 0
- joint HeadPitch: axis 0 1 0 -> 0 1.0 0; child HeadPitch_link -> Head; limit lower=-0.6720 upper=0.5149 effort=30 velocity=3.0 -> lower=-0.671952 upper=0.514872 effort=1.532 velocity=7.19407; parent HeadYaw_link -> Neck
- joint HeadYaw: axis 0 0 1 -> 0 0 1.0; child HeadYaw_link -> Neck; limit lower=-2.0857 upper=2.0857 effort=30 velocity=3.0 -> lower=-2.08567 upper=2.08567 effort=1.547 velocity=8.26797
- joint LAnklePitch: axis 0 1 0 -> 0 1.0 0; child LAnklePitch_link -> LAnklePitch; limit lower=-1.186448 upper=0.922747 effort=30 velocity=3.0 -> lower=-1.18944 upper=0.922581 effort=3.023 velocity=6.40239; origin xyz=0 0 -0.10290 rpy=0 0 0 -> xyz=0 0 -0.1029 rpy=0 0 0; parent LKneePitch_link -> LTibia
- joint LAnkleRoll: axis 1 0 0 -> 1.0 0 0; child LAnkleRoll_link -> l_ankle; limit lower=-0.769001 upper=0.397880 effort=30 velocity=3.0 -> lower=-0.397761 upper=0.768992 effort=3.348 velocity=4.16174; parent LAnklePitch_link -> LAnklePitch
- joint LElbowRoll: axis 0 0 1 -> 0 0 1.0; child LElbowRoll_link -> LForeArm; limit lower=-1.5446 upper=-0.0349 effort=30 velocity=3.0 -> lower=-1.54462 upper=-0.0349066 effort=1.532 velocity=7.19407; parent LElbowYaw_link -> LElbow
- joint LElbowYaw: axis 1 0 0 -> 1.0 0 0; child LElbowYaw_link -> LElbow; limit lower=-2.0857 upper=2.0857 effort=30 velocity=3.0 -> lower=-2.08567 upper=2.08567 effort=1.547 velocity=8.26797; parent LShoulderRoll_link -> LBicep
- joint LHipPitch: axis 0 1 0 -> 0 1.0 0; child LHipPitch_link -> LThigh; limit lower=-1.772308 upper=0.484090 effort=30 velocity=3.0 -> lower=-1.53589 upper=0.48398 effort=3.023 velocity=6.40239; parent LHipRoll_link -> LHip
- joint LHipRoll: axis 1 0 0 -> 1.0 0 0; child LHipRoll_link -> LHip; limit lower=-0.379472 upper=0.790477 effort=30 velocity=3.0 -> lower=-0.379435 upper=0.79046 effort=3.348 velocity=4.16174; parent LHipYawPitch_link -> LPelvis
- joint LHipYawPitch: child LHipYawPitch_link -> LPelvis; limit lower=-1.145303 upper=0.740810 effort=30 velocity=3.0 -> lower=-1.14529 upper=0.740718 effort=3.348 velocity=4.16174
- joint LKneePitch: axis 0 1 0 -> 0 1.0 0; child LKneePitch_link -> LTibia; limit lower=-0.092346 upper=2.112528 effort=30 velocity=3.0 -> lower=-0.0923279 upper=2.11255 effort=3.023 velocity=6.40239; parent LHipPitch_link -> LThigh
- joint LShoulderPitch: axis 0 1 0 -> 0 1.0 0; child LShoulderPitch_link -> LShoulder; limit lower=-2.0857 upper=2.0857 effort=30 velocity=3.0 -> lower=-2.08567 upper=2.08567 effort=1.329 velocity=8.26797
- joint LShoulderRoll: axis 0 0 1 -> 0 0 1.0; child LShoulderRoll_link -> LBicep; limit lower=-0.3142 upper=1.3265 effort=30 velocity=3.0 -> lower=-0.314159 upper=1.32645 effort=1.7835 velocity=7.19407; parent LShoulderPitch_link -> LShoulder
- joint LWristYaw: axis 1 0 0 -> 1.0 0 0; child LWristYaw_link -> l_wrist; limit lower=-1.8238 upper=1.8238 effort=30 velocity=3.0 -> lower=-1.82387 upper=1.82387 effort=0.4075 velocity=24.6229; parent LElbowRoll_link -> LForeArm
- joint RAnklePitch: axis 0 1 0 -> 0 1.0 0; child RAnklePitch_link -> RAnklePitch; limit lower=-1.186448 upper=0.922747 effort=30 velocity=3.0 -> lower=-1.1863 upper=0.932006 effort=3.0226 velocity=6.40239; origin xyz=0 0 -0.10290 rpy=0 0 0 -> xyz=0 0 -0.1029 rpy=0 0 0; parent RKneePitch_link -> RTibia
- joint RAnkleRoll: axis 1 0 0 -> 1.0 0 0; child RAnkleRoll_link -> r_ankle; limit lower=-0.388676 upper=0.785875 effort=30 velocity=3.0 -> lower=-0.768992 upper=0.397761 effort=3.348 velocity=4.16174; parent RAnklePitch_link -> RAnklePitch
- joint RElbowRoll: axis 0 0 1 -> 0 0 1.0; child RElbowRoll_link -> RForeArm; limit lower=0.0349 upper=1.5446 effort=30 velocity=3.0 -> lower=0.0349066 upper=1.54462 effort=1.532 velocity=7.19407; parent RElbowYaw_link -> RElbow
- joint RElbowYaw: axis 1 0 0 -> 1.0 0 0; child RElbowYaw_link -> RElbow; limit lower=-2.0857 upper=2.0857 effort=30 velocity=3.0 -> lower=-2.08567 upper=2.08567 effort=1.547 velocity=8.26797; parent RShoulderRoll_link -> RBicep
- joint RHipPitch: axis 0 1 0 -> 0 1.0 0; child RHipPitch_link -> RThigh; limit lower=-1.772308 upper=0.484090 effort=30 velocity=3.0 -> lower=-1.53589 upper=0.48398 effort=3.0226 velocity=6.40239; parent RHipRoll_link -> RHip
- joint RHipRoll: axis 1 0 0 -> 1.0 0 0; child RHipRoll_link -> RHip; limit lower=-0.738321 upper=0.414754 effort=30 velocity=3.0 -> lower=-0.79046 upper=0.379435 effort=3.348 velocity=4.16174; parent RHipYawPitch_link -> RPelvis
- joint RHipYawPitch: child RHipYawPitch_link -> RPelvis; limit lower=-1.145303 upper=0.740810 effort=30 velocity=3.0 -> lower=-1.14529 upper=0.740718 effort=3.348 velocity=4.16174; mimic joint=LHipYawPitch multiplier=1 offset=0 -> joint=LHipYawPitch multiplier=1.0 offset=0
- joint RKneePitch: axis 0 1 0 -> 0 1.0 0; child RKneePitch_link -> RTibia; limit lower=-0.092346 upper=2.112528 effort=30 velocity=3.0 -> lower=-0.0923279 upper=2.11255 effort=3.0226 velocity=6.40239; parent RHipPitch_link -> RThigh
- joint RShoulderPitch: axis 0 1 0 -> 0 1.0 0; child RShoulderPitch_link -> RShoulder; limit lower=-2.0857 upper=2.0857 effort=30 velocity=3.0 -> lower=-2.08567 upper=2.08567 effort=1.329 velocity=8.26797
- joint RShoulderRoll: axis 0 0 1 -> 0 0 1.0; child RShoulderRoll_link -> RBicep; limit lower=-1.3265 upper=0.3142 effort=30 velocity=3.0 -> lower=-1.32645 upper=0.314159 effort=1.783 velocity=7.19407; parent RShoulderPitch_link -> RShoulder
- joint RWristYaw: axis 1 0 0 -> 1.0 0 0; child RWristYaw_link -> r_wrist; limit lower=-1.8238 upper=1.8238 effort=30 velocity=3.0 -> lower=-1.82387 upper=1.82387 effort=0.4075 velocity=24.6229; parent RElbowRoll_link -> RForeArm
- joint gaze_joint: origin xyz=0.0539 0 0.05 -> xyz=0.05871 0 0.06364 rpy=0 0 0; parent HeadPitch_link -> Head
