Commit message: Fix FSR link collision names
Changed the name of the collision tags on the .xacro files for Gazebo
simulation on 'naoGazebo.xacro', which did not match the actual collision
names due to a known sdformat bug (Issue #113).

File: nao_description/urdf/naoV40_generated_urdf/naoGazebo.xacro (robot description, xacro)
@@ -3,5 +3,5 @@
     <!-- MACROS FOR DISABLE LINKS -->
 	<xacro:property name="PI" value="3.14159265359" />
-    <xacro:macro name="DisabledLinks" params="side side_small">
+<!--     <xacro:macro name="DisabledLinks" params="side side_small">
         <plugin name="${side}Finger11_link" filename="libroboticsgroup_gazebo_disable_link_plugin.so">
             <link>${side}Finger11_link</link>
@@ -31,8 +31,8 @@
             <link>${side_small}_gripper</link>
         </plugin>
-    </xacro:macro>
+    </xacro:macro> -->
     <!-- MACROS FOR MIMIC JOINTS -->
     <!-- Fingers -->
-    <xacro:macro name="FingerMimics" params="side num">
+<!--     <xacro:macro name="FingerMimics" params="side num">
         <plugin name="mimic_${side}Finger${num}1" filename="libroboticsgroup_gazebo_mimic_joint_plugin.so">
             <joint>${side}Hand</joint>
@@ -53,7 +53,7 @@
             <offset>${PI/4}</offset>
         </plugin>
-    </xacro:macro>
+    </xacro:macro> -->
     <!-- Thumbs -->
-    <xacro:macro name="ThumbMimics" params="side">
+<!--     <xacro:macro name="ThumbMimics" params="side">
         <plugin name="${side}Thumb1" filename="libroboticsgroup_gazebo_mimic_joint_plugin.so">
             <joint>${side}Hand</joint>
@@ -68,5 +68,5 @@
             <offset>${PI/4}</offset>
         </plugin>
-    </xacro:macro>
+    </xacro:macro> -->
     <!-- GAZEBO ROS CONTROL AND IMU PLUGIN -->
     <gazebo>
@@ -111,5 +111,5 @@
             <offset>0.0</offset>
         </plugin> -->
-        <xacro:FingerMimics side="L" num="1"/>
+<!--         <xacro:FingerMimics side="L" num="1"/>
         <xacro:FingerMimics side="L" num="2"/>
         <xacro:FingerMimics side="R" num="1"/>
@@ -118,5 +118,5 @@
         <xacro:ThumbMimics side="R"/>
         <xacro:DisabledLinks side="L" side_small="l"/>
-        <xacro:DisabledLinks side="R" side_small="r"/>
+        <xacro:DisabledLinks side="R" side_small="r"/> -->
     </gazebo>
     <!-- END OF GAZEBO ROS CONTROL PLUGIN -->
@@ -238,5 +238,5 @@
     </gazebo>
 -->
-    <gazebo reference="LFinger11_link">
+<!--     <gazebo reference="LFinger11_link">
         <mu1>0.5</mu1>
         <mu2>0.5</mu2>
@@ -285,5 +285,5 @@
         <selfCollide>false</selfCollide>
         <turnGravityOff>true</turnGravityOff>
-    </gazebo>
+    </gazebo> -->
     <gazebo reference="LPelvis">
         <mu1>0.5</mu1>
@@ -364,5 +364,5 @@
     <minDepth>0.003</minDepth>
   </gazebo>
-    <gazebo reference="RFinger11_link">
+<!--     <gazebo reference="RFinger11_link">
         <mu1>0.5</mu1>
         <mu2>0.5</mu2>
@@ -411,5 +411,5 @@
         <selfCollide>false</selfCollide>
         <turnGravityOff>true</turnGravityOff>
-    </gazebo>
+    </gazebo> -->
 <!--
         RGB CAMERAS: Working
@@ -553,11 +553,11 @@
 -->
 <gazebo reference="RFsrFL_frame">
-  <mu1>0.5</mu1>
+<!--   <mu1>0.5</mu1>
   <mu2>0.5</mu2>
   <selfCollide>false</selfCollide>
-  <turnGravityOff>false</turnGravityOff>
-  <fdir1>1 0 0</fdir1>
+  <turnGravityOff>false</turnGravityOff> -->
+<!--   <fdir1>1 0 0</fdir1>
   <maxVel>0.1</maxVel>
-  <minDepth>0.003</minDepth>
+  <minDepth>0.003</minDepth> -->
   <sensor name="RFsrFL" type="contact">
     <always_on>1</always_on>
@@ -565,5 +565,5 @@
     <visualize>false</visualize>
     <contact>
-      <collision>RFsrFL_frame_collision</collision>
+      <collision>r_ankle_fixed_joint_lump__RFsrFL_frame_collision_1</collision>
     </contact>
     <plugin filename="libgazebo_ros_bumper.so" name="gazebo_nao_RFsrFL">
@@ -588,5 +588,5 @@
     <visualize>false</visualize>
     <contact>
-      <collision>RFsrFR_frame_collision</collision>
+      <collision>r_ankle_fixed_joint_lump__RFsrFR_frame_collision_2</collision>
     </contact>
     <plugin filename="libgazebo_ros_bumper.so" name="gazebo_nao_RFsrFR">
@@ -611,5 +611,5 @@
     <visualize>false</visualize>
     <contact>
-      <collision>RFsrRL_frame_collision</collision>
+      <collision>r_ankle_fixed_joint_lump__RFsrRL_frame_collision_3</collision>
     </contact>
     <plugin filename="libgazebo_ros_bumper.so" name="gazebo_nao_RFsrRL">
@@ -634,5 +634,5 @@
     <visualize>false</visualize>
     <contact>
-      <collision>RFsrRR_frame_collision</collision>
+      <collision>r_ankle_fixed_joint_lump__RFsrRR_frame_collision_4</collision>
     </contact>
     <plugin filename="libgazebo_ros_bumper.so" name="gazebo_nao_RFsrRR">
@@ -657,5 +657,5 @@
     <visualize>false</visualize>
     <contact>
-      <collision>LFsrFL_frame_collision</collision>
+      <collision>l_ankle_fixed_joint_lump__LFsrFL_frame_collision_1</collision>
     </contact>
     <plugin filename="libgazebo_ros_bumper.so" name="gazebo_nao_LFsrFL">
@@ -676,12 +676,13 @@
   <minDepth>0.003</minDepth>
   <sensor name="LFsrFR" type="contact">
-    <always_on>1</always_on>
+    <always_on>true</always_on>
     <update_rate>20</update_rate>
     <visualize>false</visualize>
     <contact>
-      <collision>LFsrFR_frame_collision</collision>
+      <collision>l_ankle_fixed_joint_lump__LFsrFR_frame_collision_2</collision>
     </contact>
     <plugin filename="libgazebo_ros_bumper.so" name="gazebo_nao_ros_bumper">
       <robotNamespace>nao_robot</robotNamespace>
+      <update_rate>20</update_rate>
       <alwaysOn>true</alwaysOn>
       <bumperTopicName>FSR/LFoot/FrontRight</bumperTopicName>
@@ -703,5 +704,5 @@
     <visualize>false</visualize>
     <contact>
-      <collision>LFsrRL_frame_collision</collision>
+      <collision>l_ankle_fixed_joint_lump__LFsrRL_frame_collision_3</collision>
     </contact>
     <plugin filename="libgazebo_ros_bumper.so" name="gazebo_nao_ros_bumper">
@@ -726,5 +727,5 @@
     <visualize>false</visualize>
     <contact>
-      <collision>LFsrRR_frame_collision</collision>
+      <collision>l_ankle_fixed_joint_lump__LFsrRR_frame_collision_4</collision>
     </contact>
     <plugin filename="libgazebo_ros_bumper.so" name="gazebo_nao_ros_bumper">
