Commit message: Update link/joint nomenclature

File: nao_description/urdf/naoV50_generated_urdf/nao.urdf (robot description, URDF)
Before this commit: robot NaoH25V50, 79 links, 78 joints
Links:
- removed link LAnklePitch
- removed link RAnklePitch
- removed link l_ankle
- removed link l_sole
- removed link r_ankle
- removed link r_sole
- added link LAnkle, mass 0.13416; collision mesh filename=package://nao_meshes/meshes/V40/LAnklePitch_0.10.stl scale=0.1 0.1 0.1; visual mesh filename=package://nao_meshes/meshes/V40/LAnklePitch.dae scale=0.1 0.1 0.1
- added link LFoot, mass 0.17184; collision mesh filename=package://nao_meshes/meshes/V40/LAnkleRoll_0.10.stl scale=0.1 0.1 0.1; visual mesh filename=package://nao_meshes/meshes/V40/LAnkleRoll.dae scale=0.1 0.1 0.1
- added link LFootSole
- added link RAnkle, mass 0.13416; collision mesh filename=package://nao_meshes/meshes/V40/RAnklePitch_0.10.stl scale=0.1 0.1 0.1; visual mesh filename=package://nao_meshes/meshes/V40/RAnklePitch.dae scale=0.1 0.1 0.1
- added link RFoot, mass 0.17184; collision mesh filename=package://nao_meshes/meshes/V40/RAnkleRoll_0.10.stl scale=0.1 0.1 0.1; visual mesh filename=package://nao_meshes/meshes/V40/RAnkleRoll.dae scale=0.1 0.1 0.1
- added link RFootSole
Joints:
- joint LAnklePitch: child LAnklePitch -> LAnkle
- joint LAnkleRoll: child l_ankle -> LFoot; parent LAnklePitch -> LAnkle
- joint LFoot/Bumper/Left_sensor_fixedjoint: parent l_ankle -> LFoot
- joint LFoot/Bumper/Right_sensor_fixedjoint: parent l_ankle -> LFoot
- joint LFoot/FSR/FrontLeft_sensor_fixedjoint: parent l_ankle -> LFoot
- joint LFoot/FSR/FrontRight_sensor_fixedjoint: parent l_ankle -> LFoot
- joint LFoot/FSR/RearLeft_sensor_fixedjoint: parent l_ankle -> LFoot
- joint LFoot/FSR/RearRight_sensor_fixedjoint: parent l_ankle -> LFoot
- joint LLeg_effector_fixedjoint: child l_sole -> LFootSole; parent l_ankle -> LFoot
- joint RAnklePitch: child RAnklePitch -> RAnkle
- joint RAnkleRoll: child r_ankle -> RFoot; parent RAnklePitch -> RAnkle
- joint RFoot/Bumper/Left_sensor_fixedjoint: parent r_ankle -> RFoot
- joint RFoot/Bumper/Right_sensor_fixedjoint: parent r_ankle -> RFoot
- joint RFoot/FSR/FrontLeft_sensor_fixedjoint: parent r_ankle -> RFoot
- joint RFoot/FSR/FrontRight_sensor_fixedjoint: parent r_ankle -> RFoot
- joint RFoot/FSR/RearLeft_sensor_fixedjoint: parent r_ankle -> RFoot
- joint RFoot/FSR/RearRight_sensor_fixedjoint: parent r_ankle -> RFoot
- joint RHand: origin xyz=0.05775 0 -0.01213 rpy=0 0 0 -> xyz=0.05775 0 -0.01231 rpy=0 0 0
- joint RLeg_effector_fixedjoint: child r_sole -> RFootSole; parent r_ankle -> RFoot

File: nao_description/urdf/naoV50_generated_urdf/naoGazebo.xacro (robot description, xacro)
@@ -310,5 +310,5 @@
         <turnGravityOff>false</turnGravityOff>
     </gazebo>
- <gazebo reference="LAnklePitch">
+ <gazebo reference="LAnkle">
     <mu1>0.5</mu1>
     <mu2>0.5</mu2>
@@ -316,5 +316,5 @@
     <turnGravityOff>false</turnGravityOff>
   </gazebo>
-  <gazebo reference="l_ankle">
+  <gazebo reference="LFoot">
     <mu1>0.5</mu1>
     <mu2>0.5</mu2>
@@ -349,5 +349,5 @@
       <turnGravityOff>false</turnGravityOff>
   </gazebo>
- <gazebo reference="RAnklePitch">
+ <gazebo reference="RAnkle">
     <mu1>0.5</mu1>
     <mu2>0.5</mu2>
@@ -355,5 +355,5 @@
     <turnGravityOff>false</turnGravityOff>
   </gazebo>
-  <gazebo reference="r_ankle">
+  <gazebo reference="RFoot">
     <mu1>0.5</mu1>
     <mu2>0.5</mu2>

File: nao_description/urdf/naoV50_generated_urdf/nao_legs.xacro (robot description, xacro)
@@ -66,10 +66,10 @@
 	<joint name="LAnklePitch" type="revolute">
 		<parent link="LTibia"/>
-		<child link="LAnklePitch"/>
+		<child link="LAnkle"/>
 		<origin rpy="0 0 0" xyz="0 0 -0.1029"/>
 		<axis xyz="0 1.0 0"/>
 		<limit effort="3.023" lower="-1.18944" upper="0.922581" velocity="6.40239"/>
 	</joint>
-	<link name="LAnklePitch">
+	<link name="LAnkle">
 		<inertial>
 			<mass value="0.13416"/>
@@ -77,14 +77,14 @@
 			<origin rpy="0 0 0" xyz="0.00045 0.00029 0.00685"/>
 		</inertial>
-		<xacro:insert_visu_LAnklePitch/>
+		<xacro:insert_visu_LAnkle/>
 	</link>
 	<joint name="LAnkleRoll" type="revolute">
-		<parent link="LAnklePitch"/>
-		<child link="l_ankle"/>
+		<parent link="LAnkle"/>
+		<child link="LFoot"/>
 		<origin rpy="0 0 0" xyz="0 0 0"/>
 		<axis xyz="1.0 0 0"/>
 		<limit effort="3.348" lower="-0.397761" upper="0.768992" velocity="4.16174"/>
 	</joint>
-	<link name="l_ankle">
+	<link name="LFoot">
 		<inertial>
 			<mass value="0.17184"/>
@@ -92,13 +92,13 @@
 			<origin rpy="0 0 0" xyz="0.02542 0.0033 -0.03239"/>
 		</inertial>
-		<xacro:insert_visu_l_ankle/>
+		<xacro:insert_visu_LFoot/>
 	</link>
 	<joint name="LLeg_effector_fixedjoint" type="fixed">
-		<parent link="l_ankle"/>
-		<child link="l_sole"/>
+		<parent link="LFoot"/>
+		<child link="LFootSole"/>
 		<origin rpy="0 0 0" xyz="0 0 -0.04511"/>
 		<axis xyz="0 0 0"/>
 	</joint>
-	<link name="l_sole"/>
+	<link name="LFootSole"/>
 	<joint name="RHipYawPitch" type="revolute">
 		<parent link="torso"/>
@@ -164,10 +164,10 @@
 	<joint name="RAnklePitch" type="revolute">
 		<parent link="RTibia"/>
-		<child link="RAnklePitch"/>
+		<child link="RAnkle"/>
 		<origin rpy="0 0 0" xyz="0 0 -0.1029"/>
 		<axis xyz="0 1.0 0"/>
 		<limit effort="3.0226" lower="-1.1863" upper="0.932006" velocity="6.40239"/>
 	</joint>
-	<link name="RAnklePitch">
+	<link name="RAnkle">
 		<inertial>
 			<mass value="0.13416"/>
@@ -175,14 +175,14 @@
 			<origin rpy="0 0 0" xyz="0.00045 -0.00029 0.00685"/>
 		</inertial>
-		<xacro:insert_visu_RAnklePitch/>
+		<xacro:insert_visu_RAnkle/>
 	</link>
 	<joint name="RAnkleRoll" type="revolute">
-		<parent link="RAnklePitch"/>
-		<child link="r_ankle"/>
+		<parent link="RAnkle"/>
+		<child link="RFoot"/>
 		<origin rpy="0 0 0" xyz="0 0 0"/>
 		<axis xyz="1.0 0 0"/>
 		<limit effort="3.348" lower="-0.768992" upper="0.397761" velocity="4.16174"/>
 	</joint>
-	<link name="r_ankle">
+	<link name="RFoot">
 		<inertial>
 			<mass value="0.17184"/>
@@ -190,12 +190,12 @@
 			<origin rpy="0 0 0" xyz="0.02542 -0.0033 -0.03239"/>
 		</inertial>
-		<xacro:insert_visu_r_ankle/>
+		<xacro:insert_visu_RFoot/>
 	</link>
 	<joint name="RLeg_effector_fixedjoint" type="fixed">
-		<parent link="r_ankle"/>
-		<child link="r_sole"/>
+		<parent link="RFoot"/>
+		<child link="RFootSole"/>
 		<origin rpy="0 0 0" xyz="0 0 -0.04511"/>
 		<axis xyz="0 0 0"/>
 	</joint>
-	<link name="r_sole"/>
+	<link name="RFootSole"/>
 </robot>

File: nao_description/urdf/naoV50_generated_urdf/nao_sensors.xacro (robot description, xacro)
@@ -6,5 +6,5 @@
 	<link name="LFootBumperRight_frame"/>
 	<joint name="LFoot/Bumper/Right_sensor_fixedjoint" type="fixed">
-		<parent link="l_ankle"/>
+		<parent link="LFoot"/>
 		<child link="LFootBumperRight_frame"/>
 		<origin rpy="0 0 0" xyz="0.0876 -0.014 -0.0353"/>
@@ -24,5 +24,5 @@
 	</link>
 	<joint name="RFoot/FSR/RearLeft_sensor_fixedjoint" type="fixed">
-		<parent link="r_ankle"/>
+		<parent link="RFoot"/>
 		<child link="RFsrRL_frame"/>
 		<origin rpy="0 0 0" xyz="-0.03025 0.0191 -0.04511"/>
@@ -48,5 +48,5 @@
 	</link>
 	<joint name="RFoot/FSR/RearRight_sensor_fixedjoint" type="fixed">
-		<parent link="r_ankle"/>
+		<parent link="RFoot"/>
 		<child link="RFsrRR_frame"/>
 		<origin rpy="0 0 0" xyz="-0.02965 -0.0299 -0.04511"/>
@@ -66,5 +66,5 @@
 	</link>
 	<joint name="LFoot/FSR/FrontRight_sensor_fixedjoint" type="fixed">
-		<parent link="l_ankle"/>
+		<parent link="LFoot"/>
 		<child link="LFsrFR_frame"/>
 		<origin rpy="0 0 0" xyz="0.07025 -0.0231 -0.04511"/>
@@ -80,5 +80,5 @@
 	<link name="RFootBumperRight_frame"/>
 	<joint name="RFoot/Bumper/Right_sensor_fixedjoint" type="fixed">
-		<parent link="r_ankle"/>
+		<parent link="RFoot"/>
 		<child link="RFootBumperRight_frame"/>
 		<origin rpy="0 0 0" xyz="0.0876 -0.019 -0.0353"/>
@@ -98,5 +98,5 @@
 	</link>
 	<joint name="RFoot/FSR/FrontRight_sensor_fixedjoint" type="fixed">
-		<parent link="r_ankle"/>
+		<parent link="RFoot"/>
 		<child link="RFsrFR_frame"/>
 		<origin rpy="0 0 0" xyz="0.07025 -0.0299 -0.04511"/>
@@ -116,5 +116,5 @@
 	</link>
 	<joint name="LFoot/FSR/RearRight_sensor_fixedjoint" type="fixed">
-		<parent link="l_ankle"/>
+		<parent link="LFoot"/>
 		<child link="LFsrRR_frame"/>
 		<origin rpy="0 0 0" xyz="-0.02965 -0.0191 -0.04511"/>
@@ -137,5 +137,5 @@
 	<link name="RFootBumperLeft_frame"/>
 	<joint name="RFoot/Bumper/Left_sensor_fixedjoint" type="fixed">
-		<parent link="r_ankle"/>
+		<parent link="RFoot"/>
 		<child link="RFootBumperLeft_frame"/>
 		<origin rpy="0 0 0" xyz="0.0876 0.014 -0.0353"/>
@@ -176,5 +176,5 @@
 	</link>
 	<joint name="RFoot/FSR/FrontLeft_sensor_fixedjoint" type="fixed">
-		<parent link="r_ankle"/>
+		<parent link="RFoot"/>
 		<child link="RFsrFL_frame"/>
 		<origin rpy="0 0 0" xyz="0.07025 0.0231 -0.04511"/>
@@ -201,5 +201,5 @@
 	</link>
 	<joint name="LFoot/FSR/FrontLeft_sensor_fixedjoint" type="fixed">
-		<parent link="l_ankle"/>
+		<parent link="LFoot"/>
 		<child link="LFsrFL_frame"/>
 		<origin rpy="0 0 0" xyz="0.07025 0.0299 -0.04511"/>
@@ -219,5 +219,5 @@
 	</link>
 	<joint name="LFoot/FSR/RearLeft_sensor_fixedjoint" type="fixed">
-		<parent link="l_ankle"/>
+		<parent link="LFoot"/>
 		<child link="LFsrRL_frame"/>
 		<origin rpy="0 0 0" xyz="-0.03025 0.0299 -0.04511"/>
@@ -302,5 +302,5 @@
 	<link name="LFootBumperLeft_frame"/>
 	<joint name="LFoot/Bumper/Left_sensor_fixedjoint" type="fixed">
-		<parent link="l_ankle"/>
+		<parent link="LFoot"/>
 		<child link="LFootBumperLeft_frame"/>
 		<origin rpy="0 0 0" xyz="0.0876 0.019 -0.0353"/>

File: nao_description/urdf/naoV50_generated_urdf/nao_visual_collisions.xacro (robot description, xacro)
@@ -656,5 +656,5 @@
 		</xacro:if>
 	</xacro:macro>
-	<xacro:macro name="insert_visu_LAnklePitch">
+	<xacro:macro name="insert_visu_LAnkle">
 		<xacro:unless value="${meshes_installed}"/>
 		<xacro:if value="${meshes_installed}">
@@ -690,5 +690,5 @@
 		</xacro:if>
 	</xacro:macro>
-	<xacro:macro name="insert_visu_RAnklePitch">
+	<xacro:macro name="insert_visu_RAnkle">
 		<xacro:unless value="${meshes_installed}"/>
 		<xacro:if value="${meshes_installed}">
@@ -738,5 +738,5 @@
 		</xacro:if>
 	</xacro:macro>
-	<xacro:macro name="insert_visu_r_ankle">
+	<xacro:macro name="insert_visu_RFoot">
 		<xacro:unless value="${meshes_installed}">
 			<visual>
@@ -769,5 +769,5 @@
 		</xacro:if>
 	</xacro:macro>
-	<xacro:macro name="insert_visu_l_ankle">
+	<xacro:macro name="insert_visu_LFoot">
 		<xacro:unless value="${meshes_installed}">
 			<visual>
