Commit message: Add simplified model with fixed hip yaw joints and update FSR position

File: nao_description/urdf/naoV50_handless_nohipyaw_generated_urdf/nao_sensors.xacro (robot description, xacro)
@@ -34,5 +34,6 @@
 		<child link="RFsrRL_frame"/>
       <!-- <origin rpy="0 0 0" xyz="-0.03025 0.0191 -0.04511"/> -->
-      <origin rpy="0 0 0" xyz="-0.03025 0.0191 -0.04261"/>
+      <!-- <origin rpy="0 0 0" xyz="-0.03025 0.0191 -0.04261"/> -->
+      <origin rpy="0 0 0" xyz="-0.03025 0.0191 -0.04261"/>  <!-- offset to ensure ground contact -->
 		<axis xyz="0 0 0"/>
 	</joint>
@@ -66,5 +67,6 @@
 		<child link="RFsrRR_frame"/>
 			<!-- <origin rpy="0 0 0" xyz="-0.03025 -0.0299 -0.04511"/> -->
-			<origin rpy="0 0 0" xyz="-0.03025 -0.0299 -0.04261"/>
+			<!-- <origin rpy="0 0 0" xyz="-0.03025 -0.0299 -0.04261"/>  -->
+			<origin rpy="0 0 0" xyz="-0.03025 -0.0299 -0.04261"/>  <!-- offset to ensure ground contact -->
 		<axis xyz="0 0 0"/>
 	</joint>
@@ -92,5 +94,6 @@
 		<child link="LFsrFR_frame"/>
 			<!-- <origin rpy="0 0 0" xyz="0.07025 -0.0231 -0.04511"/> -->
-			<origin rpy="0 0 0" xyz="0.07025 -0.0231 -0.04261"/>
+			<!-- <origin rpy="0 0 0" xyz="0.07025 -0.0231 -0.04261"/> -->
+			<origin rpy="0 0 0" xyz="0.07025 -0.0231 -0.04261"/>  <!-- offset to ensure ground contact -->
 		<axis xyz="0 0 0"/>
 	</joint>
@@ -125,5 +128,6 @@
 		<child link="RFsrFR_frame"/>
 		<!-- <origin rpy="0 0 0" xyz="0.07025 -0.0299 -0.04511"/> -->
-		<origin rpy="0 0 0" xyz="0.07025 -0.0299 -0.04261"/>
+		<!-- <origin rpy="0 0 0" xyz="0.07025 -0.0299 -0.04261"/> -->
+		<origin rpy="0 0 0" xyz="0.07025 -0.0299 -0.04261"/>  <!-- offset to ensure ground contact -->
 		<axis xyz="0 0 0"/>
 	</joint>
@@ -151,5 +155,6 @@
 		<child link="LFsrRR_frame"/>
 			<!-- <origin rpy="0 0 0" xyz="-0.03025 -0.0191 -0.04511"/> -->
-			<origin rpy="0 0 0" xyz="-0.03025 -0.0191 -0.04261"/>
+			<!-- <origin rpy="0 0 0" xyz="-0.03025 -0.0191 -0.04261"/> -->
+			<origin rpy="0 0 0" xyz="-0.03025 -0.0191 -0.04261"/>  <!-- offset to ensure ground contact -->
 		<axis xyz="0 0 0"/>
 	</joint>
@@ -206,5 +211,6 @@
 		<child link="RFsrFL_frame"/>
 			<!-- <origin rpy="0 0 0" xyz="0.07025 0.0231 -0.04511"/> -->
-			<origin rpy="0 0 0" xyz="0.07025 0.0231 -0.04261"/>
+			<!-- <origin rpy="0 0 0" xyz="0.07025 0.0231 -0.04261"/> -->
+			<origin rpy="0 0 0" xyz="0.07025 0.0231 -0.04261"/>  <!-- offset to ensure ground contact -->
 		<axis xyz="0 0 0"/>
 	</joint>
@@ -239,5 +245,6 @@
 		<child link="LFsrFL_frame"/>
 			<!-- <origin rpy="0 0 0" xyz="0.07025 0.0299 -0.04511"/> -->
-			<origin rpy="0 0 0" xyz="0.07025 0.0299 -0.04261"/>
+			<!-- <origin rpy="0 0 0" xyz="0.07025 0.0299 -0.04261"/> -->
+			<origin rpy="0 0 0" xyz="0.07025 0.0299 -0.04261"/>  <!-- offset to ensure ground contact -->
 		<axis xyz="0 0 0"/>
 	</joint>
@@ -265,5 +272,6 @@
 		<child link="LFsrRL_frame"/>
 			<!-- <origin rpy="0 0 0" xyz="-0.03025 0.0299 -0.04511"/> -->
-			<origin rpy="0 0 0" xyz="-0.03025 0.0299 -0.04261"/>
+			<!-- <origin rpy="0 0 0" xyz="-0.03025 0.0299 -0.04261"/> -->
+			<origin rpy="0 0 0" xyz="-0.03025 0.0299 -0.04261"/>  <!-- offset to ensure ground contact -->
 		<axis xyz="0 0 0"/>
 	</joint>
